File: electronics/nuclone_small_libmcull_tester/nuclone_small_libmcull_tester.kicad_pcb (KiCad board)
At the start: 2 copper layers, 50 x 50 mm, 75 parts, among them J1 Conn_02x04_Odd_Even, J10 Conn_02x03_Odd_Even, J11 Conn_02x04_Odd_Even, J2 Conn_02x04_Odd_Even, J3 nuclone_small_left, J4 nuclone_small_right, J5 FTDI_PINS_1X06, J6 DevBoardUartInput, J7 Conn_02x02_Odd_Even, J8 Conn_02x02_Odd_Even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

Commit message: updated footprints and versionnumber
Other:
- board text removed: "RC_out1"

Commit message: small fixes, preparing for production
Parts:
- N2: value V20230915 -> V20240426
Other:
- board text added: "RC_out1"
Changed lines of the file:
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@@
     (property "ki_description" "Generic connector, double row, 02x04, odd/even pin numbering scheme (row 1 odd numbers, row 2 even numbers), script generated (kicad-library-utils/schlib/autogen/connector/)")
     (property "ki_keywords" "connector")
-    (attr through_hole exclude_from_pos_files exclude_from_bom)
+    (attr through_hole exclude_from_pos_files)
     (fp_text reference "J9" (at 0 -3.5 -90) (layer "F.SilkS")
         (effects (font (size 1 1) (thickness 0.15)))
@@
     (property "ki_description" "Generic connector, double row, 02x03, odd/even pin numbering scheme (row 1 odd numbers, row 2 even numbers), script generated (kicad-library-utils/schlib/autogen/connector/)")
     (property "ki_keywords" "connector")
-    (attr through_hole exclude_from_pos_files exclude_from_bom)
+    (attr through_hole exclude_from_pos_files)
     (fp_text reference "J10" (at 4 3.9 180) (layer "F.SilkS")
         (effects (font (size 1 1) (thickness 0.15)))
@@
     (property "ki_description" "Generic connector, double row, 02x04, odd/even pin numbering scheme (row 1 odd numbers, row 2 even numbers), script generated (kicad-library-utils/schlib/autogen/connector/)")
     (property "ki_keywords" "connector")
-    (attr through_hole exclude_from_pos_files exclude_from_bom)
+    (attr through_hole exclude_from_pos_files)
     (fp_text reference "J1" (at 5.8 0) (layer "F.SilkS")
         (effects (font (size 1 1) (thickness 0.15)))
@@
     (property "ki_description" "Generic connector, double row, 02x02, odd/even pin numbering scheme (row 1 odd numbers, row 2 even numbers), script generated (kicad-library-utils/schlib/autogen/connector/)")
     (property "ki_keywords" "connector")
-    (attr through_hole exclude_from_pos_files exclude_from_bom)
+    (attr through_hole exclude_from_pos_files)
     (fp_text reference "J8" (at 3.275 0) (layer "F.SilkS")
         (effects (font (size 1 1) (thickness 0.15)))
@@
     (property "ki_description" "Generic connector, double row, 02x02, odd/even pin numbering scheme (row 1 odd numbers, row 2 even numbers), script generated (kicad-library-utils/schlib/autogen/connector/)")
     (property "ki_keywords" "connector")
-    (attr through_hole exclude_from_pos_files exclude_from_bom)
+    (attr through_hole exclude_from_pos_files)
     (fp_text reference "J7" (at 3.275 0) (layer "F.SilkS")
         (effects (font (size 1 1) (thickness 0.15)))
@@
     (property "ki_description" "Generic connector, double row, 02x04, odd/even pin numbering scheme (row 1 odd numbers, row 2 even numbers), script generated (kicad-library-utils/schlib/autogen/connector/)")
     (property "ki_keywords" "connector")
-    (attr through_hole exclude_from_pos_files exclude_from_bom)
+    (attr through_hole exclude_from_pos_files)
     (fp_text reference "J11" (at 0 -3.5 -90) (layer "F.SilkS")
         (effects (font (size 1 1) (thickness 0.15)))
@@
     (property "Sheetfile" "nuclone_small_libmcull_tester.kicad_sch")
     (property "Sheetname" "")
-    (attr exclude_from_pos_files exclude_from_bom)
+    (attr exclude_from_pos_files)
     (fp_text reference "J5" (at 8.5 0 180) (layer "F.SilkS")
         (effects (font (size 1 1) (thickness 0.15)))
@@
     (property "ki_description" "Generic connector, double row, 02x04, odd/even pin numbering scheme (row 1 odd numbers, row 2 even numbers), script generated (kicad-library-utils/schlib/autogen/connector/)")
     (property "ki_keywords" "connector")
-    (attr through_hole exclude_from_pos_files exclude_from_bom)
+    (attr through_hole exclude_from_pos_files)
     (fp_text reference "J2" (at 5.8 0) (layer "F.SilkS")
         (effects (font (size 1 1) (thickness 0.15)))
@@
         (effects (font (size 1 1) (thickness 0.15)) (justify mirror))
     )
-    (fp_text value "V20230915" (at 0 0.1) (layer "B.SilkS")
+    (fp_text value "V20240426" (at 0 0.1) (layer "B.SilkS")
         (effects (font (size 0.8 0.8) (thickness 0.15)) (justify mirror))
     )
@@
     (effects (font (size 1 1) (thickness 0.15)) (justify left bottom))
   )
+  (gr_text "RC_out1" (at 92 89) (layer "F.SilkS")
+    (effects (font (size 1 1) (thickness 0.15)) (justify left bottom))
+  )

Commit message: added numbering of test gpio's
Other:
- board text added: "PIN5"
- board text added: "PIN6"
- board text added: "PIN7"
- board text added: "PIN8"
Changed lines of the file:
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@@
     (effects (font (size 1 1) (thickness 0.15)) (justify left bottom))
   )
-  (gr_text "PIN4" (at 92 85.1) (layer "F.SilkS")
+  (gr_text "PIN8" (at 92 85.1) (layer "F.SilkS")
     (effects (font (size 1 1) (thickness 0.15)) (justify left bottom))
   )
@@
     (effects (font (size 1 1) (thickness 0.15)) (justify left bottom))
   )
-  (gr_text "PIN1" (at 92 77.4) (layer "F.SilkS")
+  (gr_text "PIN2" (at 92 77.4) (layer "F.SilkS")
     (effects (font (size 1 1) (thickness 0.15)) (justify left bottom))
   )
-  (gr_text "PIN2" (at 74.3 80) (layer "F.SilkS")
+  (gr_text "PIN3" (at 74.3 80) (layer "F.SilkS")
     (effects (font (size 1 1) (thickness 0.15)) (justify left bottom))
   )
@@
     (effects (font (size 1 1) (thickness 0.15)) (justify left bottom))
   )
-  (gr_text "PIN3" (at 74.3 82.5) (layer "F.SilkS")
+  (gr_text "PIN5" (at 74.3 82.5) (layer "F.SilkS")
     (effects (font (size 1 1) (thickness 0.15)) (justify left bottom))
   )
-  (gr_text "PIN4" (at 74.3 85.1) (layer "F.SilkS")
+  (gr_text "PIN7" (at 74.3 85.1) (layer "F.SilkS")
     (effects (font (size 1 1) (thickness 0.15)) (justify left bottom))
   )
-  (gr_text "PIN2" (at 92 80) (layer "F.SilkS")
+  (gr_text "PIN4" (at 92 80) (layer "F.SilkS")
     (effects (font (size 1 1) (thickness 0.15)) (justify left bottom))
   )
-  (gr_text "PIN3" (at 92 82.5) (layer "F.SilkS")
+  (gr_text "PIN6" (at 92 82.5) (layer "F.SilkS")
     (effects (font (size 1 1) (thickness 0.15)) (justify left bottom))
   )
