File: electronics/nuclone_small_libmcull_tester/nuclone_small_libmcull_tester.kicad_sch (KiCad schematic)
At the start: 75 parts, among them J1 Conn_02x04_Odd_Even, J10 Conn_02x03_Odd_Even, J11 Conn_02x04_Odd_Even, J2 Conn_02x04_Odd_Even, J3 nuclone_small_left, J4 nuclone_small_right, J5 FTDI_PINS_1X06, J6 DevBoardUartInput, J7 Conn_02x02_Odd_Even, J8 Conn_02x02_Odd_Even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

Commit message: updated footprints and versionnumber
Parts:
- N2: value V20230915 -> V20240422
Changed lines of the file:
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@@
       (effects (font (size 1.524 1.524)) (justify left))
     )
-    (property "Value" "V20230915" (at 17.78 182.88 0)
+    (property "Value" "V20240422" (at 17.78 182.88 0)
       (effects (font (size 1.524 1.524)) (justify left))
     )

Commit message: small fixes, preparing for production
Parts:
- N2: value V20240422 -> V20240426
Changed lines of the file:
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@@
       (effects (font (size 1.524 1.524)) (justify left))
     )
-    (property "Value" "V20240422" (at 17.78 182.88 0)
+    (property "Value" "V20240426" (at 17.78 182.88 0)
       (effects (font (size 1.524 1.524)) (justify left))
     )

Commit message: preparation for production
Parts:
- N2: value V20240426 -> V20240712
Changed lines of the file:
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@@
       (effects (font (size 1.524 1.524)) (justify left))
     )
-    (property "Value" "V20240426" (at 17.78 182.88 0)
+    (property "Value" "V20240712" (at 17.78 182.88 0)
       (effects (font (size 1.524 1.524)) (justify left))
     )
